File: hub_imu.kicad_pcb (KiCad board)
At the start: 2 copper layers, 21 x 14.4 mm, 19 parts, among them J1 USB 1x4 P2.54, J2 SWD 2x3 P1.27, U1 STM32F042F6P6, U2 BNO055, U3 AP2112K-3.3

Commit message: Use JLCPCB basic parts; add "JLCPCB Part #" field to all parts
- Add a "JLCPCB Part #" field to every symbol/footprint, using codes
  confirmed as basic via JLCPCB's parts API (C1525, C52923, C23733,
  C25744, C25900, C11702, C2286, C5446). U1, U2, J1 and J2 are left
  blank (ICs not basic; headers hand-soldered).
- U3: AP2112K-3.3 (SOT-23-5, extended) -> XC6206P332MR (SOT-23-3, basic
  C5446). Pinout per Torex datasheet: 1 VSS, 2 VOUT, 3 VIN; the EN tie
  is removed. Rotated 180 deg so VIN faces J1/C1, and the corner re-routed.
- D1: 0402 LED -> 0603 red KT-0603R (basic C2286). R5/D1 shifted
  0.8 mm left so the cathode gets its own GND via.
- Refill pours, re-stitch; final DRC 0 errors / 0 unconnected.
- README: parts table with JLCPCB numbers, new U3/D1.

Co-Authored-By: Claude Opus 5.5 <noreply@anthropic.com>
Parts:
- D1: footprint LED_SMD:LED_0402_1005Metric -> LED_SMD:LED_0603_1608Metric
- U3: value AP2112K-3.3 -> XC6206P332MR; footprint Package_TO_SOT_SMD:SOT-23-5 -> Package_TO_SOT_SMD:SOT-23-3
- moved D1 0.81 mm to (87.9, 92.8)
- moved R5 0.80 mm to (85.5, 92.8)
- turned U3 to 180 degrees
Connections:
- U3 pad 1: +5V -> GND
- U3 pad 2: GND -> +3V3
Routing:
- net +5V: track 9.92 -> 6.41 mm
- net /STATUS_LED: track 6.85 -> 6.05 mm
- net GND: track 20.5 -> 21.3 mm, vias 17 -> 16

Commit message: Board: EweFeel 1.0 back silkscreen, J1/J2 DNP, mask clearance 0.005 mm
Co-Authored-By: Claude Opus 5.5 <noreply@anthropic.com>
Other:
- board text added: "EweFeel 1.0 9/2026"
- board text added: "sdg"
Changed lines of the file:
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@@
 		(sheetname "/")
 		(sheetfile "hub_imu.kicad_sch")
-		(attr through_hole)
+		(attr through_hole dnp)
 		(fp_line
 			(start -1.38 9)
@@
 		(sheetname "/")
 		(sheetfile "hub_imu.kicad_sch")
-		(attr through_hole)
+		(attr through_hole dnp)
 		(fp_line
 			(start 2.45 -0.745)
@@
 		(layer "Edge.Cuts")
 	)
+	(gr_text "sdg"
+		(at 75 94 0)
+		(layer "B.SilkS")
+		(effects
+			(font
+				(size 1 1)
+				(thickness 0.1)
+			)
+			(justify left bottom mirror)
+		)
+	)
+	(gr_text "EweFeel 1.0\n9/2026"
+		(at 88 87 0)
+		(layer "B.SilkS")
+		(effects
+			(font
+				(size 1 1)
+				(thickness 0.1)
+			)
+			(justify left bottom mirror)
+		)
+	)
 	(segment
